Commit message: Update init

File: config/we_r2_arm.urdf.xacro (robot description, xacro)
@@ -5,5 +5,5 @@
     <origin rpy="0 0 0" xyz="0 0 0"/>
     <geometry>
-      <mesh filename="package://we_r2_moveit_config/config/bin_stl/base_link_m-binary.stl"/>
+      <mesh filename="package://we_r2_moveit_config/config/bin_stl/stl/base_link_9_11_1.stl"/>
     </geometry>
     <material name="silver">
@@ -14,5 +14,6 @@
     <origin rpy="0 0 0" xyz="0 0 0"/>
     <geometry>
-        <mesh filename="package://we_r2_moveit_config/config/col_stl/collision_base_link.stl"/>
+      <!-- don't forget about collision  -->
+        <mesh filename="package://we_r2_moveit_config/config/col_stl/collision_base_link_test.stl"/>
     </geometry>
   </collision>
@@ -27,5 +28,5 @@
     <origin rpy="0 0 0" xyz="0.035775 0.074529 -0.366958"/>
     <geometry>
-      <mesh filename="package://we_r2_moveit_config/config/bin_stl/Forearm__1_m-binary.stl"/>
+      <mesh filename="package://we_r2_moveit_config/config/bin_stl/stl/arm_2.stl"/>
     </geometry>
     <material name="silver">
@@ -36,5 +37,5 @@
     <origin rpy="0 0 0" xyz="0.035775 0.074529 -0.366958"/>
     <geometry>
-        <mesh filename="package://we_r2_moveit_config/config/col_stl/collision_forearm.stl"/>
+        <mesh filename="package://we_r2_moveit_config/config/col_stl/collision_forearm_test.stl"/>
     </geometry>
   </collision>
@@ -49,5 +50,5 @@
     <origin rpy="0 0 0" xyz="0.024453 0.074942 -0.544758"/>
     <geometry>
-      <mesh filename="package://we_r2_moveit_config/config/bin_stl/wrist_1__1_m-binary.stl"/>
+      <mesh filename="package://we_r2_moveit_config/config/bin_stl/stl/wrist_link_1.stl"/>
     </geometry>
     <material name="silver">
@@ -71,5 +72,5 @@
     <origin rpy="0 0 0" xyz="-0.012324 0.074585 -0.163809"/>
     <geometry>
-      <mesh filename="package://we_r2_moveit_config/config/bin_stl/upper_arm__1_m-binary.stl"/>
+      <mesh filename="package://we_r2_moveit_config/config/bin_stl/stl/arm_1.stl"/>
     </geometry>
     <material name="silver">
@@ -93,5 +94,5 @@
     <origin rpy="0 0 0" xyz="-0.000666 0.07459 -0.106659"/>
     <geometry>
-      <mesh filename="package://we_r2_moveit_config/config/bin_stl/shoulder__1_m-binary.stl"/>
+      <mesh filename="package://we_r2_moveit_config/config/bin_stl/stl/shoulder_actuator_1.stl"/>
     </geometry>
     <material name="silver">
@@ -115,5 +116,5 @@
     <origin rpy="0 0 0" xyz="-0.002217 0.074916 -0.576213"/>
     <geometry>
-      <mesh filename="package://we_r2_moveit_config/config/bin_stl/wrist_2__1_m-binary.stl"/>
+      <mesh filename="package://we_r2_moveit_config/config/bin_stl/stl/wrist_link_2.stl"/>
     </geometry>
     <material name="silver">
@@ -150,10 +151,10 @@
   </collision>
 </link>
-<joint name="joint2" type="continuous">
-  <origin rpy="0 0 0" xyz="-0.048099 5.6e-05 0.203149"/>
+<joint name="joint2" type="revolute">
+  <origin rpy="0 0 0" xyz="-0.00192 5.6e-05 0.229559"/>
   <parent link="upper_arm__1"/>
   <child link="Forearm__1"/>
   <axis xyz="-0.01 1.7e-05 0.0"/>
-  <limit effort="100" velocity="0.5"/>
+  <limit effort="100" velocity="0.5" upper="1.57" lower="-1.57"/>
 </joint>
 <transmission name="joint2_tran">
@@ -167,10 +168,10 @@
   </actuator>
 </transmission>
-<joint name="joint3" type="continuous">
-  <origin rpy="0 0 0" xyz="0.011322 -0.000413 0.1778"/>
+<joint name="joint3" type="revolute">
+  <origin rpy="0 0 0" xyz="0.011322 -0.000113 0.2142"/>
   <parent link="Forearm__1"/>
   <child link="wrist_1__1"/>
   <axis xyz="0.01 -1.7e-05 -0.0"/>
-  <limit effort="100" velocity="0.5"/>
+  <limit effort="100" velocity="0.5" upper="1.57" lower="-1.57" />
 </joint>
 <transmission name="joint3_tran">
@@ -184,10 +185,10 @@
   </actuator>
 </transmission>
-<joint name="joint1" type="continuous">
-  <origin rpy="0 0 0" xyz="0.011658 5e-06 0.05715"/>
+<joint name="joint1" type="revolute">
+  <origin rpy="0 0 0" xyz="0.065458 5e-06 0.03505"/>
   <parent link="shoulder__1"/>
   <child link="upper_arm__1"/>
   <axis xyz="0.01 -1.7e-05 0.0"/>
-  <limit effort="100" velocity="0.5"/>
+  <limit effort="100" velocity="0.5" upper="1.57" lower="-1.57" />
 </joint>
 <transmission name="joint1_tran">
@@ -201,10 +202,10 @@
   </actuator>
 </transmission>
-<joint name="joint0" type="continuous">
-  <origin rpy="0 0 0" xyz="0.000666 -0.07459 0.106659"/>
+<joint name="joint0" type="revolute">
+  <origin rpy="0 0 0" xyz="0.000666 -0.07459 0.0302246"/>
   <parent link="base_link"/>
   <child link="shoulder__1"/>
   <axis xyz="0.0 0.0 0.01"/>
-  <limit effort="100" velocity="0.5"/>
+  <limit effort="100" velocity="0.5" upper="1.57" lower="-1.57" />
 </joint>
 <transmission name="joint0_tran">
@@ -218,10 +219,11 @@
   </actuator>
 </transmission>
-<joint name="joint4" type="continuous">
-  <origin rpy="0 0 0" xyz="0.02667 2.6e-05 0.031455"/>
+<joint name="joint4" type="revolute">
+  <origin rpy="0 0 0" xyz="0.0441 2.6e-05 0.031555"/>
+  <!-- <origin rpy="0 0 0" xyz="0.0267067 2.6e-05 0.030455"/> -->
   <parent link="wrist_1__1"/>
   <child link="wrist_2__1"/>
   <axis xyz="0.0 2.2e-05 0.01"/>
-  <limit effort="100" velocity="0.5"/>
+  <limit effort="100" velocity="0.5" upper="1.57" lower="-1.57" />
 </joint>
 <transmission name="joint4_tran">
@@ -235,10 +237,10 @@
   </actuator>
 </transmission>
-<joint name="joint5" type="continuous">
-  <origin rpy="0 0 0" xyz="-0.000148 0.031513 0.0266"/>
+<joint name="joint5" type="revolute">
+  <origin rpy="0 0 0" xyz="-0.000148 0.031513 0.0459"/>
   <parent link="wrist_2__1"/>
   <child link="end_effector_link__1"/>
   <axis xyz="-4.7e-05 0.01 -2.2e-05"/>
-  <limit effort="100" velocity="0.5"/>
+  <limit effort="100" velocity="0.5" upper="1.57" lower="-1.57" />
 </joint>
 <transmission name="joint5_tran">

Commit message: Create detector of aruco tf

File: config/we_r2_arm.urdf.xacro (robot description, xacro)
@@ -152,5 +152,5 @@
 </link>
 <joint name="joint2" type="revolute">
-  <origin rpy="0 0 0" xyz="-0.00192 5.6e-05 0.229559"/>
+  <origin rpy="0 0 0" xyz="-0.00192 5.6e-05 0.228559"/>
   <parent link="upper_arm__1"/>
   <child link="Forearm__1"/>

Commit message: Update conf

File: config/we_r2_arm.urdf.xacro (robot description, xacro)
@@ -151,10 +151,10 @@
   </collision>
 </link>
-<joint name="joint2" type="revolute">
+<joint name="joint2" type="continuous">
   <origin rpy="0 0 0" xyz="-0.00192 5.6e-05 0.228559"/>
   <parent link="upper_arm__1"/>
   <child link="Forearm__1"/>
   <axis xyz="-0.01 1.7e-05 0.0"/>
-  <limit effort="100" velocity="0.5" upper="1.57" lower="-1.57"/>
+  <limit effort="100" velocity="0.5"/>
 </joint>
 <transmission name="joint2_tran">
@@ -168,10 +168,10 @@
   </actuator>
 </transmission>
-<joint name="joint3" type="revolute">
+<joint name="joint3" type="continuous">
   <origin rpy="0 0 0" xyz="0.011322 -0.000113 0.2142"/>
   <parent link="Forearm__1"/>
   <child link="wrist_1__1"/>
   <axis xyz="0.01 -1.7e-05 -0.0"/>
-  <limit effort="100" velocity="0.5" upper="1.57" lower="-1.57" />
+  <limit effort="100" velocity="0.5"/>
 </joint>
 <transmission name="joint3_tran">
@@ -185,10 +185,10 @@
   </actuator>
 </transmission>
-<joint name="joint1" type="revolute">
+<joint name="joint1" type="continuous">
   <origin rpy="0 0 0" xyz="0.065458 5e-06 0.03505"/>
   <parent link="shoulder__1"/>
   <child link="upper_arm__1"/>
   <axis xyz="0.01 -1.7e-05 0.0"/>
-  <limit effort="100" velocity="0.5" upper="1.57" lower="-1.57" />
+  <limit effort="100" velocity="0.5"/>
 </joint>
 <transmission name="joint1_tran">
@@ -202,10 +202,10 @@
   </actuator>
 </transmission>
-<joint name="joint0" type="revolute">
+<joint name="joint0" type="continuous">
   <origin rpy="0 0 0" xyz="0.000666 -0.07459 0.0302246"/>
   <parent link="base_link"/>
   <child link="shoulder__1"/>
   <axis xyz="0.0 0.0 0.01"/>
-  <limit effort="100" velocity="0.5" upper="1.57" lower="-1.57" />
+  <limit effort="100" velocity="0.5" />
 </joint>
 <transmission name="joint0_tran">
@@ -219,5 +219,5 @@
   </actuator>
 </transmission>
-<joint name="joint4" type="revolute">
+<joint name="joint4" type="continuous">
   <origin rpy="0 0 0" xyz="0.0441 2.6e-05 0.031555"/>
   <!-- <origin rpy="0 0 0" xyz="0.0267067 2.6e-05 0.030455"/> -->
@@ -225,5 +225,5 @@
   <child link="wrist_2__1"/>
   <axis xyz="0.0 2.2e-05 0.01"/>
-  <limit effort="100" velocity="0.5" upper="1.57" lower="-1.57" />
+  <limit effort="100" velocity="0.5" />
 </joint>
 <transmission name="joint4_tran">
@@ -237,10 +237,10 @@
   </actuator>
 </transmission>
-<joint name="joint5" type="revolute">
+<joint name="joint5" type="continuous">
   <origin rpy="0 0 0" xyz="-0.000148 0.031513 0.0459"/>
   <parent link="wrist_2__1"/>
   <child link="end_effector_link__1"/>
   <axis xyz="-4.7e-05 0.01 -2.2e-05"/>
-  <limit effort="100" velocity="0.5" upper="1.57" lower="-1.57" />
+  <limit effort="100" velocity="0.5" />
 </joint>
 <transmission name="joint5_tran">

Commit message: Update urdf

File: config/we_r2_arm.urdf.xacro (robot description, xacro)
@@ -151,10 +151,10 @@
   </collision>
 </link>
-<joint name="joint2" type="continuous">
+<joint name="joint2" type="revolute">
   <origin rpy="0 0 0" xyz="-0.00192 5.6e-05 0.228559"/>
   <parent link="upper_arm__1"/>
   <child link="Forearm__1"/>
   <axis xyz="-0.01 1.7e-05 0.0"/>
-  <limit effort="100" velocity="0.5"/>
+  <limit effort="100" velocity="0.5" upper="2.27" lower="-2.27" />
 </joint>
 <transmission name="joint2_tran">
@@ -168,10 +168,10 @@
   </actuator>
 </transmission>
-<joint name="joint3" type="continuous">
+<joint name="joint3" type="revolute">
   <origin rpy="0 0 0" xyz="0.011322 -0.000113 0.2142"/>
   <parent link="Forearm__1"/>
   <child link="wrist_1__1"/>
   <axis xyz="0.01 -1.7e-05 -0.0"/>
-  <limit effort="100" velocity="0.5"/>
+  <limit effort="100" velocity="0.5" upper="2.27" lower="-2.27"/>
 </joint>
 <transmission name="joint3_tran">
@@ -185,10 +185,10 @@
   </actuator>
 </transmission>
-<joint name="joint1" type="continuous">
+<joint name="joint1" type="revolute">
   <origin rpy="0 0 0" xyz="0.065458 5e-06 0.03505"/>
   <parent link="shoulder__1"/>
   <child link="upper_arm__1"/>
   <axis xyz="0.01 -1.7e-05 0.0"/>
-  <limit effort="100" velocity="0.5"/>
+  <limit effort="100" velocity="0.5" upper="2.27" lower="-2.27"/>
 </joint>
 <transmission name="joint1_tran">
@@ -202,10 +202,10 @@
   </actuator>
 </transmission>
-<joint name="joint0" type="continuous">
+<joint name="joint0" type="revolute">
   <origin rpy="0 0 0" xyz="0.000666 -0.07459 0.0302246"/>
   <parent link="base_link"/>
   <child link="shoulder__1"/>
   <axis xyz="0.0 0.0 0.01"/>
-  <limit effort="100" velocity="0.5" />
+  <limit effort="100" velocity="0.5" upper="2.27" lower="-2.27"/>
 </joint>
 <transmission name="joint0_tran">
@@ -219,5 +219,5 @@
   </actuator>
 </transmission>
-<joint name="joint4" type="continuous">
+<joint name="joint4" type="revolute">
   <origin rpy="0 0 0" xyz="0.0441 2.6e-05 0.031555"/>
   <!-- <origin rpy="0 0 0" xyz="0.0267067 2.6e-05 0.030455"/> -->
@@ -225,5 +225,5 @@
   <child link="wrist_2__1"/>
   <axis xyz="0.0 2.2e-05 0.01"/>
-  <limit effort="100" velocity="0.5" />
+  <limit effort="100" velocity="0.5" upper="2.27" lower="-2.27"/>
 </joint>
 <transmission name="joint4_tran">
@@ -237,10 +237,10 @@
   </actuator>
 </transmission>
-<joint name="joint5" type="continuous">
+<joint name="joint5" type="revolute">
   <origin rpy="0 0 0" xyz="-0.000148 0.031513 0.0459"/>
   <parent link="wrist_2__1"/>
   <child link="end_effector_link__1"/>
   <axis xyz="-4.7e-05 0.01 -2.2e-05"/>
-  <limit effort="100" velocity="0.5" />
+  <limit effort="100" velocity="0.5" upper="2.27" lower="-2.27"/>
 </joint>
 <transmission name="joint5_tran">

Commit message: Fix: set joint1 limits on -90/+90

File: config/we_r2_arm.urdf.xacro (robot description, xacro)
@@ -190,5 +190,5 @@
   <child link="upper_arm__1"/>
   <axis xyz="0.01 -1.7e-05 0.0"/>
-  <limit effort="100" velocity="0.5" upper="2.27" lower="-2.27"/>
+  <limit effort="100" velocity="0.5" upper="1.57" lower="-1.57"/>
 </joint>
 <transmission name="joint1_tran">

Commit message: Add new gripper model

File: config/we_r2_arm.urdf.xacro (robot description, xacro)
@@ -116,5 +116,5 @@
     <origin rpy="0 0 0" xyz="-0.002217 0.074916 -0.576213"/>
     <geometry>
-      <mesh filename="package://we_r2_moveit_config/config/bin_stl/stl/wrist_link_2.stl"/>
+      <mesh filename="package://we_r2_moveit_config/config/bin_stl/wrist_2__1_m-binar/stl/wrist_link_2.stl"/>
     </geometry>
     <material name="silver">
@@ -138,5 +138,5 @@
     <origin rpy="0 0 0" xyz="-0.002069 0.043403 -0.602813"/>
     <geometry>
-      <mesh filename="package://we_r2_moveit_config/config/bin_stl/end_effector_link__1_m-binary.stl"/>
+      <mesh filename="package://we_r2_moveit_config/config/bin_stl/stl/gripper.stl"/>
     </geometry>
     <material name="silver">

Commit message: Replacement end effector & Change gripper position

File: config/we_r2_arm.urdf.xacro (robot description, xacro)
@@ -116,5 +116,5 @@
     <origin rpy="0 0 0" xyz="-0.002217 0.074916 -0.576213"/>
     <geometry>
-      <mesh filename="package://we_r2_moveit_config/config/bin_stl/wrist_2__1_m-binar/stl/wrist_link_2.stl"/>
+      <mesh filename="package://we_r2_moveit_config/config/bin_stl/stl/wrist_link_2.stl"/>
     </geometry>
     <material name="silver">
@@ -136,5 +136,5 @@
   </inertial>
   <visual>
-    <origin rpy="0 0 0" xyz="-0.002069 0.043403 -0.602813"/>
+    <origin rpy="0 0 0" xyz="-0.114 0.043403 -0.59"/>
     <geometry>
       <mesh filename="package://we_r2_moveit_config/config/bin_stl/stl/gripper.stl"/>
@@ -147,5 +147,6 @@
     <origin rpy="0 1.5708 0" xyz="-3.800000000000027e-05 0.007937999999999994 -1.8000000000073513e-05"/>
     <geometry>
-      <cylinder length="0.05" radius="0.02"/>
+      <!-- <cylinder length="0.05" radius="0.02"/> -->
+      <mesh filename="package://we_r2_moveit_config/config/col_stl/collision_gripper.stl"/>
     </geometry>
   </collision>

Commit message: fix: remove useless stl models

File: config/we_r2_arm.urdf.xacro (robot description, xacro)
@@ -5,5 +5,5 @@
     <origin rpy="0 0 0" xyz="0 0 0"/>
     <geometry>
-      <mesh filename="package://we_r2_moveit_config/config/bin_stl/stl/base_link_9_11_1.stl"/>
+      <mesh filename="package://we_r2_moveit_config/config/bit_stl/base_link_9_11_1.stl"/>
     </geometry>
     <material name="silver">
@@ -28,5 +28,5 @@
     <origin rpy="0 0 0" xyz="0.035775 0.074529 -0.366958"/>
     <geometry>
-      <mesh filename="package://we_r2_moveit_config/config/bin_stl/stl/arm_2.stl"/>
+      <mesh filename="package://we_r2_moveit_config/config/bit_stl/arm_2.stl"/>
     </geometry>
     <material name="silver">
@@ -50,5 +50,5 @@
     <origin rpy="0 0 0" xyz="0.024453 0.074942 -0.544758"/>
     <geometry>
-      <mesh filename="package://we_r2_moveit_config/config/bin_stl/stl/wrist_link_1.stl"/>
+      <mesh filename="package://we_r2_moveit_config/config/bit_stl/wrist_link_1.stl"/>
     </geometry>
     <material name="silver">
@@ -72,5 +72,5 @@
     <origin rpy="0 0 0" xyz="-0.012324 0.074585 -0.163809"/>
     <geometry>
-      <mesh filename="package://we_r2_moveit_config/config/bin_stl/stl/arm_1.stl"/>
+      <mesh filename="package://we_r2_moveit_config/config/bit_stl/arm_1.stl"/>
     </geometry>
     <material name="silver">
@@ -94,5 +94,5 @@
     <origin rpy="0 0 0" xyz="-0.000666 0.07459 -0.106659"/>
     <geometry>
-      <mesh filename="package://we_r2_moveit_config/config/bin_stl/stl/shoulder_actuator_1.stl"/>
+      <mesh filename="package://we_r2_moveit_config/config/bit_stl/shoulder_actuator_1.stl"/>
     </geometry>
     <material name="silver">
@@ -116,5 +116,5 @@
     <origin rpy="0 0 0" xyz="-0.002217 0.074916 -0.576213"/>
     <geometry>
-      <mesh filename="package://we_r2_moveit_config/config/bin_stl/stl/wrist_link_2.stl"/>
+      <mesh filename="package://we_r2_moveit_config/config/bit_stl/wrist_link_2.stl"/>
     </geometry>
     <material name="silver">
@@ -138,5 +138,5 @@
     <origin rpy="0 0 0" xyz="-0.114 0.043403 -0.59"/>
     <geometry>
-      <mesh filename="package://we_r2_moveit_config/config/bin_stl/stl/gripper.stl"/>
+      <mesh filename="package://we_r2_moveit_config/config/bit_stl/gripper.stl"/>
     </geometry>
     <material name="silver">

Commit message: fix: repair path and set xyz for new stl models

File: config/we_r2_arm.urdf.xacro (robot description, xacro)
@@ -5,5 +5,5 @@
     <origin rpy="0 0 0" xyz="0 0 0"/>
     <geometry>
-      <mesh filename="package://we_r2_moveit_config/config/bit_stl/base_link_9_11_1.stl"/>
+      <mesh filename="package://we_r2_moveit_config/config/bin_stl/base_link_9_11_1.stl"/>
     </geometry>
     <material name="silver">
@@ -28,5 +28,5 @@
     <origin rpy="0 0 0" xyz="0.035775 0.074529 -0.366958"/>
     <geometry>
-      <mesh filename="package://we_r2_moveit_config/config/bit_stl/arm_2.stl"/>
+      <mesh filename="package://we_r2_moveit_config/config/bin_stl/arm_2.stl"/>
     </geometry>
     <material name="silver">
@@ -48,7 +48,7 @@
   </inertial>
   <visual>
-    <origin rpy="0 0 0" xyz="0.024453 0.074942 -0.544758"/>
-    <geometry>
-      <mesh filename="package://we_r2_moveit_config/config/bit_stl/wrist_link_1.stl"/>
+    <origin rpy="0 0 0" xyz="0.024453 0.074942 -0.581758"/>
+    <geometry>
+      <mesh filename="package://we_r2_moveit_config/config/bin_stl/new_wrist_link_1.stl"/>
     </geometry>
     <material name="silver">
@@ -72,5 +72,5 @@
     <origin rpy="0 0 0" xyz="-0.012324 0.074585 -0.163809"/>
     <geometry>
-      <mesh filename="package://we_r2_moveit_config/config/bit_stl/arm_1.stl"/>
+      <mesh filename="package://we_r2_moveit_config/config/bin_stl/arm_1.stl"/>
     </geometry>
     <material name="silver">
@@ -94,5 +94,5 @@
     <origin rpy="0 0 0" xyz="-0.000666 0.07459 -0.106659"/>
     <geometry>
-      <mesh filename="package://we_r2_moveit_config/config/bit_stl/shoulder_actuator_1.stl"/>
+      <mesh filename="package://we_r2_moveit_config/config/bin_stl/shoulder_actuator_1.stl"/>
     </geometry>
     <material name="silver">
@@ -114,7 +114,7 @@
   </inertial>
   <visual>
-    <origin rpy="0 0 0" xyz="-0.002217 0.074916 -0.576213"/>
-    <geometry>
-      <mesh filename="package://we_r2_moveit_config/config/bit_stl/wrist_link_2.stl"/>
+    <origin rpy="0 0 0" xyz="-0.019517 0.074916 -0.613213"/>
+    <geometry>
+      <mesh filename="package://we_r2_moveit_config/config/bin_stl/new_wrist_link_2.stl"/>
     </geometry>
     <material name="silver">
@@ -138,5 +138,5 @@
     <origin rpy="0 0 0" xyz="-0.114 0.043403 -0.59"/>
     <geometry>
-      <mesh filename="package://we_r2_moveit_config/config/bit_stl/gripper.stl"/>
+      <mesh filename="package://we_r2_moveit_config/config/bin_stl/new_gripper.stl"/>
     </geometry>
     <material name="silver">

Commit message: chore: fix the last joint

File: config/we_r2_arm.urdf.xacro (robot description, xacro)
@@ -136,5 +136,5 @@
   </inertial>
   <visual>
-    <origin rpy="0 0 0" xyz="-0.114 0.043403 -0.59"/>
+    <origin rpy="0 0 0" xyz="-0.0195 0.043403 -0.505"/>
     <geometry>
       <mesh filename="package://we_r2_moveit_config/config/bin_stl/new_gripper.stl"/>
@@ -239,5 +239,5 @@
 </transmission>
 <joint name="joint5" type="revolute">
-  <origin rpy="0 0 0" xyz="-0.000148 0.031513 0.0459"/>
+  <origin rpy="0 0 0" xyz="-0.000148 0.031513 -0.1089"/>
   <parent link="wrist_2__1"/>
   <child link="end_effector_link__1"/>
