Commit message: feat: add dirs to share

File: src/we_r2_arm_description/urdf/we_r2_arm.urdf.xacro (robot description, xacro)
@@ -2,4 +2,16 @@
 <robot xmlns:xacro="https://www.ros.org/wiki/xacro" name="we_r2_arm">
     <link name="world" />
-    <!-- TODO: links and joints -->
+    <link name="base_link">
+        <visual>
+            <origin rpy="0 0 0"  xyz="0 0 0" />
+            <geometry>
+                <mesh filename="package://we_r2_arm_description/meshes/shoulder_actuator_1.stl" scale="1 1 1" />
+            </geometry>
+        </visual>
+    </link>
+    <joint name="virtual_joint" type="fixed">
+        <parent link="world" />
+        <child link="base_link" />
+        <origin rpy="0 0 0" xyz="0 0 0" />
+    </joint>
 </robot>

Commit message: feat: add the old urdf structure so far

File: src/we_r2_arm_description/urdf/we_r2_arm.urdf.xacro (robot description, xacro)
@@ -1,3 +1,264 @@
-<?xml version="1.0"?>
+<?xml version="1.0" ?>
+<robot name="we_r2_arm" xmlns:xacro="http://www.ros.org/wiki/xacro">
+<link name="base_link">
+  <visual>
+    <origin rpy="0 0 0" xyz="0 0 0"/>
+    <geometry>
+      <mesh filename="package://we_r2_arm_description/meshes/base_link_9_11_1.stl"/>
+    </geometry>
+    <material name="silver">
+      <color rgba="1 0 0 1"/>
+    </material>
+  </visual>
+  <collision>
+    <origin rpy="0 0 0" xyz="0 0 0"/>
+    <geometry>
+      <!-- don't forget about collision  -->
+        <mesh filename="package://we_r2_moveit_config/config/col_stl/collision_base_link_test.stl"/>
+    </geometry>
+  </collision>
+</link>
+<link name="Forearm__1">
+  <inertial>
+    <origin rpy="0 0 0" xyz="-0.014792 -0.00013599999999999723 0.101354"/>
+    <mass value="0.670217"/>
+    <inertia ixx="0.004244" ixy="0.0" ixz="0.007572" iyy="0.004259" iyz="-0.007549" izz="0.000301"/>
+  </inertial>
+  <visual>
+    <origin rpy="0 0 0" xyz="0.035775 0.074529 -0.366958"/>
+    <geometry>
+      <mesh filename="package://we_r2_arm_description/meshes/arm_2.stl"/>
+    </geometry>
+    <material name="silver">
+      <color rgba="1 0 0 1"/>
+    </material>
+  </visual>
+  <collision>
+    <origin rpy="0 0 0" xyz="0.035775 0.074529 -0.366958"/>
+    <geometry>
+        <mesh filename="package://we_r2_moveit_config/config/col_stl/collision_forearm_test.stl"/>
+    </geometry>
+  </collision>
+</link>
+<link name="wrist_1__1">
+  <inertial>
+    <origin rpy="0 0 0" xyz="0.025382 -1.000000000001e-06 0.0072510000000000074"/>
+    <mass value="0.282343"/>
+    <inertia ixx="0.000154" ixy="0.0" ixz="0.011825" iyy="0.000162" iyz="-0.011831" izz="0.000133"/>
+  </inertial>
+  <visual>
+    <origin rpy="0 0 0" xyz="0.024453 0.074942 -0.581758"/>
+    <geometry>
+      <mesh filename="package://we_r2_arm_description/meshes/new_wrist_link_1.stl"/>
+    </geometry>
+    <material name="silver">
+      <color rgba="1 0 0 1"/>
+    </material>
+  </visual>
+  <collision>
+    <origin rpy="0 0 0" xyz="0.024453 0.074942 -0.544758"/>
+    <geometry>
+        <mesh filename="package://we_r2_moveit_config/config/col_stl/collision_wrist_1.stl"/>
+    </geometry>
+  </collision>
+</link>
+<link name="upper_arm__1">
+  <inertial>
+    <origin rpy="0 0 0" xyz="-0.015592 -6.1000000000005494e-05 0.20106100000000002"/>
+    <mass value="0.465826"/>
+    <inertia ixx="0.000327" ixy="0.0" ixz="0.012132" iyy="0.000496" iyz="-0.012106" izz="0.000474"/>
+  </inertial>
+  <visual>
+    <origin rpy="0 0 0" xyz="-0.012324 0.074585 -0.163809"/>
+    <geometry>
+      <mesh filename="package://we_r2_arm_description/meshes/arm_1.stl"/>
+    </geometry>
+    <material name="silver">
+      <color rgba="1 0 0 1"/>
+    </material>
+  </visual>
+  <collision>
+    <origin rpy="0 0 0" xyz="-0.012324 0.074585 -0.163809"/>
+    <geometry>
+        <mesh filename="package://we_r2_moveit_config/config/col_stl/collision_upper_arm.stl"/>
+    </geometry>
+  </collision>
+</link>
+<link name="shoulder__1">
+  <inertial>
+    <origin rpy="0 0 0" xyz="-0.019159 8.900000000000574e-05 0.04272799999999999"/>
+    <mass value="1.493039"/>
+    <inertia ixx="0.002392" ixy="2e-06" ixz="0.012495" iyy="0.002653" iyz="-0.012347" izz="0.001979"/>
+  </inertial>
+  <visual>
+    <origin rpy="0 0 0" xyz="-0.000666 0.07459 -0.106659"/>
+    <geometry>
+      <mesh filename="package://we_r2_arm_description/meshes/shoulder_actuator_1.stl"/>
+    </geometry>
+    <material name="silver">
+      <color rgba="1 0 0 1"/>
+    </material>
+  </visual>
+  <collision>
+    <origin rpy="0 0 0" xyz="-0.000666 0.07459 -0.106659"/>
+    <geometry>
+        <mesh filename="package://we_r2_moveit_config/config/col_stl/collision_shoulder.stl"/>
+    </geometry>
+  </collision>
+</link>
+<link name="wrist_2__1">
+  <inertial>
+    <origin rpy="0 0 0" xyz="-3.399999999999974e-05 0.007306999999999994 0.025361000000000078"/>
+    <mass value="0.282365"/>
+    <inertia ixx="0.000162" ixy="-0.0" ixz="0.011849" iyy="0.000133" iyz="-0.011855" izz="0.000155"/>
+  </inertial>
+  <visual>
+    <origin rpy="0 0 0" xyz="-0.019517 0.074916 -0.613213"/>
+    <geometry>
+      <mesh filename="package://we_r2_arm_description/meshes/new_wrist_link_2.stl"/>
+    </geometry>
+    <material name="silver">
+      <color rgba="1 0 0 1"/>
+    </material>
+  </visual>
+  <collision>
+    <origin rpy="0 0 0" xyz="-0.002217 0.074916 -0.576213"/>
+    <geometry>
+        <mesh filename="package://we_r2_moveit_config/config/col_stl/collision_wrist_2.stl"/>
+    </geometry>
+  </collision>
+</link>
+<link name="end_effector_link__1">
+  <inertial>
+    <origin rpy="0 0 0" xyz="-3.800000000000027e-05 0.007937999999999994 -1.8000000000073513e-05"/>
+    <mass value="0.0358"/>
+    <inertia ixx="3e-06" ixy="-0.0" ixz="0.000809" iyy="1.2e-05" iyz="-0.000809" izz="1.2e-05"/>
+  </inertial>
+  <visual>
+    <origin rpy="0 0 0" xyz="-0.0195 0.043403 -0.505"/>
+    <geometry>
+      <mesh filename="package://we_r2_arm_description/meshes/new_gripper.stl"/>
+    </geometry>
+    <material name="silver">
+      <color rgba="1 0 0 1"/>
+    </material>
+  </visual>
+  <collision>
+    <origin rpy="0 1.5708 0" xyz="-3.800000000000027e-05 0.007937999999999994 -1.8000000000073513e-05"/>
+    <geometry>
+      <!-- <cylinder length="0.05" radius="0.02"/> -->
+      <mesh filename="package://we_r2_moveit_config/config/col_stl/collision_gripper.stl"/>
+    </geometry>
+  </collision>
+</link>
+<joint name="joint2" type="revolute">
+  <origin rpy="0 0 0" xyz="-0.00192 5.6e-05 0.228559"/>
+  <parent link="upper_arm__1"/>
+  <child link="Forearm__1"/>
+  <axis xyz="-0.01 1.7e-05 0.0"/>
+  <limit effort="100" velocity="0.5" upper="2.27" lower="-2.27" />
+</joint>
+<transmission name="joint2_tran">
+  <type>transmission_interface/SimpleTransmission</type>
+  <joint name="joint2">
+    <hardwareInterface>PositionJointInterface</hardwareInterface>
+  </joint>
+  <actuator name="joint2_actr">
+    <hardwareInterface>PositionJointInterface</hardwareInterface>
+    <mechanicalReduction>1</mechanicalReduction>
+  </actuator>
+</transmission>
+<joint name="joint3" type="revolute">
+  <origin rpy="0 0 0" xyz="0.011322 -0.000113 0.2142"/>
+  <parent link="Forearm__1"/>
+  <child link="wrist_1__1"/>
+  <axis xyz="0.01 -1.7e-05 -0.0"/>
+  <limit effort="100" velocity="0.5" upper="2.27" lower="-2.27"/>
+</joint>
+<transmission name="joint3_tran">
+  <type>transmission_interface/SimpleTransmission</type>
+  <joint name="joint3">
+    <hardwareInterface>PositionJointInterface</hardwareInterface>
+  </joint>
+  <actuator name="joint3_actr">
+    <hardwareInterface>PositionJointInterface</hardwareInterface>
+    <mechanicalReduction>1</mechanicalReduction>
+  </actuator>
+</transmission>
+<joint name="joint1" type="revolute">
+  <origin rpy="0 0 0" xyz="0.065458 5e-06 0.03505"/>
+  <parent link="shoulder__1"/>
+  <child link="upper_arm__1"/>
+  <axis xyz="0.01 -1.7e-05 0.0"/>
+  <limit effort="100" velocity="0.5" upper="1.57" lower="-1.57"/>
+</joint>
+<transmission name="joint1_tran">
+  <type>transmission_interface/SimpleTransmission</type>
+  <joint name="joint1">
+    <hardwareInterface>PositionJointInterface</hardwareInterface>
+  </joint>
+  <actuator name="joint1_actr">
+    <hardwareInterface>PositionJointInterface</hardwareInterface>
+    <mechanicalReduction>1</mechanicalReduction>
+  </actuator>
+</transmission>
+<joint name="joint0" type="revolute">
+  <origin rpy="0 0 0" xyz="0.000666 -0.07459 0.0302246"/>
+  <parent link="base_link"/>
+  <child link="shoulder__1"/>
+  <axis xyz="0.0 0.0 0.01"/>
+  <limit effort="100" velocity="0.5" upper="2.27" lower="-2.27"/>
+</joint>
+<transmission name="joint0_tran">
+  <type>transmission_interface/SimpleTransmission</type>
+  <joint name="joint0">
+    <hardwareInterface>PositionJointInterface</hardwareInterface>
+  </joint>
+  <actuator name="joint0_actr">
+    <hardwareInterface>PositionJointInterface</hardwareInterface>
+    <mechanicalReduction>1</mechanicalReduction>
+  </actuator>
+</transmission>
+<joint name="joint4" type="revolute">
+  <origin rpy="0 0 0" xyz="0.0441 2.6e-05 0.031555"/>
+  <!-- <origin rpy="0 0 0" xyz="0.0267067 2.6e-05 0.030455"/> -->
+  <parent link="wrist_1__1"/>
+  <child link="wrist_2__1"/>
+  <axis xyz="0.0 2.2e-05 0.01"/>
+  <limit effort="100" velocity="0.5" upper="2.27" lower="-2.27"/>
+</joint>
+<transmission name="joint4_tran">
+  <type>transmission_interface/SimpleTransmission</type>
+  <joint name="joint4">
+    <hardwareInterface>PositionJointInterface</hardwareInterface>
+  </joint>
+  <actuator name="joint4_actr">
+    <hardwareInterface>PositionJointInterface</hardwareInterface>
+    <mechanicalReduction>1</mechanicalReduction>
+  </actuator>
+</transmission>
+<joint name="joint5" type="revolute">
+  <origin rpy="0 0 0" xyz="-0.000148 0.031513 -0.1089"/>
+  <parent link="wrist_2__1"/>
+  <child link="end_effector_link__1"/>
+  <axis xyz="-4.7e-05 0.01 -2.2e-05"/>
+  <limit effort="100" velocity="0.5" upper="2.27" lower="-2.27"/>
+</joint>
+<transmission name="joint5_tran">
+  <type>transmission_interface/SimpleTransmission</type>
+  <joint name="joint5">
+    <hardwareInterface>PositionJointInterface</hardwareInterface>
+  </joint>
+  <actuator name="joint5_actr">
+    <hardwareInterface>PositionJointInterface</hardwareInterface>
+    <mechanicalReduction>1</mechanicalReduction>
+  </actuator>
+</transmission>
+<gazebo>
+  <plugin filename="libgazebo_ros_control.so" name="control"/>
+</gazebo>
+</robot>
+<!-- TODO: rewrite urdf xacro using code below -->
+<!-- <?xml version="1.0"?>
 <robot xmlns:xacro="https://www.ros.org/wiki/xacro" name="we_r2_arm">
     <link name="world" />
@@ -15,3 +276,3 @@
         <origin rpy="0 0 0" xyz="0 0 0" />
     </joint>
-</robot>
+</robot> -->

Commit message: feat: create display launch file & display rviz

File: src/we_r2_arm_description/urdf/we_r2_arm.urdf.xacro (robot description, xacro)
@@ -259,20 +259,2 @@
 </gazebo>
 </robot>
-<!-- TODO: rewrite urdf xacro using code below -->
-<!-- <?xml version="1.0"?>
-<robot xmlns:xacro="https://www.ros.org/wiki/xacro" name="we_r2_arm">
-    <link name="world" />
-    <link name="base_link">
-        <visual>
-            <origin rpy="0 0 0"  xyz="0 0 0" />
-            <geometry>
-                <mesh filename="package://we_r2_arm_description/meshes/shoulder_actuator_1.stl" scale="1 1 1" />
-            </geometry>
-        </visual>
-    </link>
-    <joint name="virtual_joint" type="fixed">
-        <parent link="world" />
-        <child link="base_link" />
-        <origin rpy="0 0 0" xyz="0 0 0" />
-    </joint>
-</robot> -->

Commit message: feat: start reworking urdf xacro

File: src/we_r2_arm_description/urdf/we_r2_arm.urdf.xacro (robot description, xacro)
@@ -1,260 +1,17 @@
-<?xml version="1.0" ?>
-<robot name="we_r2_arm" xmlns:xacro="http://www.ros.org/wiki/xacro">
-<link name="base_link">
-  <visual>
-    <origin rpy="0 0 0" xyz="0 0 0"/>
-    <geometry>
-      <mesh filename="package://we_r2_arm_description/meshes/base_link_9_11_1.stl"/>
-    </geometry>
-    <material name="silver">
-      <color rgba="1 0 0 1"/>
-    </material>
-  </visual>
-  <collision>
-    <origin rpy="0 0 0" xyz="0 0 0"/>
-    <geometry>
-      <!-- don't forget about collision  -->
-        <mesh filename="package://we_r2_moveit_config/config/col_stl/collision_base_link_test.stl"/>
-    </geometry>
-  </collision>
-</link>
-<link name="Forearm__1">
-  <inertial>
-    <origin rpy="0 0 0" xyz="-0.014792 -0.00013599999999999723 0.101354"/>
-    <mass value="0.670217"/>
-    <inertia ixx="0.004244" ixy="0.0" ixz="0.007572" iyy="0.004259" iyz="-0.007549" izz="0.000301"/>
-  </inertial>
-  <visual>
-    <origin rpy="0 0 0" xyz="0.035775 0.074529 -0.366958"/>
-    <geometry>
-      <mesh filename="package://we_r2_arm_description/meshes/arm_2.stl"/>
-    </geometry>
-    <material name="silver">
-      <color rgba="1 0 0 1"/>
-    </material>
-  </visual>
-  <collision>
-    <origin rpy="0 0 0" xyz="0.035775 0.074529 -0.366958"/>
-    <geometry>
-        <mesh filename="package://we_r2_moveit_config/config/col_stl/collision_forearm_test.stl"/>
-    </geometry>
-  </collision>
-</link>
-<link name="wrist_1__1">
-  <inertial>
-    <origin rpy="0 0 0" xyz="0.025382 -1.000000000001e-06 0.0072510000000000074"/>
-    <mass value="0.282343"/>
-    <inertia ixx="0.000154" ixy="0.0" ixz="0.011825" iyy="0.000162" iyz="-0.011831" izz="0.000133"/>
-  </inertial>
-  <visual>
-    <origin rpy="0 0 0" xyz="0.024453 0.074942 -0.581758"/>
-    <geometry>
-      <mesh filename="package://we_r2_arm_description/meshes/new_wrist_link_1.stl"/>
-    </geometry>
-    <material name="silver">
-      <color rgba="1 0 0 1"/>
-    </material>
-  </visual>
-  <collision>
-    <origin rpy="0 0 0" xyz="0.024453 0.074942 -0.544758"/>
-    <geometry>
-        <mesh filename="package://we_r2_moveit_config/config/col_stl/collision_wrist_1.stl"/>
-    </geometry>
-  </collision>
-</link>
-<link name="upper_arm__1">
-  <inertial>
-    <origin rpy="0 0 0" xyz="-0.015592 -6.1000000000005494e-05 0.20106100000000002"/>
-    <mass value="0.465826"/>
-    <inertia ixx="0.000327" ixy="0.0" ixz="0.012132" iyy="0.000496" iyz="-0.012106" izz="0.000474"/>
-  </inertial>
-  <visual>
-    <origin rpy="0 0 0" xyz="-0.012324 0.074585 -0.163809"/>
-    <geometry>
-      <mesh filename="package://we_r2_arm_description/meshes/arm_1.stl"/>
-    </geometry>
-    <material name="silver">
-      <color rgba="1 0 0 1"/>
-    </material>
-  </visual>
-  <collision>
-    <origin rpy="0 0 0" xyz="-0.012324 0.074585 -0.163809"/>
-    <geometry>
-        <mesh filename="package://we_r2_moveit_config/config/col_stl/collision_upper_arm.stl"/>
-    </geometry>
-  </collision>
-</link>
-<link name="shoulder__1">
-  <inertial>
-    <origin rpy="0 0 0" xyz="-0.019159 8.900000000000574e-05 0.04272799999999999"/>
-    <mass value="1.493039"/>
-    <inertia ixx="0.002392" ixy="2e-06" ixz="0.012495" iyy="0.002653" iyz="-0.012347" izz="0.001979"/>
-  </inertial>
-  <visual>
-    <origin rpy="0 0 0" xyz="-0.000666 0.07459 -0.106659"/>
-    <geometry>
-      <mesh filename="package://we_r2_arm_description/meshes/shoulder_actuator_1.stl"/>
-    </geometry>
-    <material name="silver">
-      <color rgba="1 0 0 1"/>
-    </material>
-  </visual>
-  <collision>
-    <origin rpy="0 0 0" xyz="-0.000666 0.07459 -0.106659"/>
-    <geometry>
-        <mesh filename="package://we_r2_moveit_config/config/col_stl/collision_shoulder.stl"/>
-    </geometry>
-  </collision>
-</link>
-<link name="wrist_2__1">
-  <inertial>
-    <origin rpy="0 0 0" xyz="-3.399999999999974e-05 0.007306999999999994 0.025361000000000078"/>
-    <mass value="0.282365"/>
-    <inertia ixx="0.000162" ixy="-0.0" ixz="0.011849" iyy="0.000133" iyz="-0.011855" izz="0.000155"/>
-  </inertial>
-  <visual>
-    <origin rpy="0 0 0" xyz="-0.019517 0.074916 -0.613213"/>
-    <geometry>
-      <mesh filename="package://we_r2_arm_description/meshes/new_wrist_link_2.stl"/>
-    </geometry>
-    <material name="silver">
-      <color rgba="1 0 0 1"/>
-    </material>
-  </visual>
-  <collision>
-    <origin rpy="0 0 0" xyz="-0.002217 0.074916 -0.576213"/>
-    <geometry>
-        <mesh filename="package://we_r2_moveit_config/config/col_stl/collision_wrist_2.stl"/>
-    </geometry>
-  </collision>
-</link>
-<link name="end_effector_link__1">
-  <inertial>
-    <origin rpy="0 0 0" xyz="-3.800000000000027e-05 0.007937999999999994 -1.8000000000073513e-05"/>
-    <mass value="0.0358"/>
-    <inertia ixx="3e-06" ixy="-0.0" ixz="0.000809" iyy="1.2e-05" iyz="-0.000809" izz="1.2e-05"/>
-  </inertial>
-  <visual>
-    <origin rpy="0 0 0" xyz="-0.0195 0.043403 -0.505"/>
-    <geometry>
-      <mesh filename="package://we_r2_arm_description/meshes/new_gripper.stl"/>
-    </geometry>
-    <material name="silver">
-      <color rgba="1 0 0 1"/>
-    </material>
-  </visual>
-  <collision>
-    <origin rpy="0 1.5708 0" xyz="-3.800000000000027e-05 0.007937999999999994 -1.8000000000073513e-05"/>
-    <geometry>
-      <!-- <cylinder length="0.05" radius="0.02"/> -->
-      <mesh filename="package://we_r2_moveit_config/config/col_stl/collision_gripper.stl"/>
-    </geometry>
-  </collision>
-</link>
-<joint name="joint2" type="revolute">
-  <origin rpy="0 0 0" xyz="-0.00192 5.6e-05 0.228559"/>
-  <parent link="upper_arm__1"/>
-  <child link="Forearm__1"/>
-  <axis xyz="-0.01 1.7e-05 0.0"/>
-  <limit effort="100" velocity="0.5" upper="2.27" lower="-2.27" />
-</joint>
-<transmission name="joint2_tran">
-  <type>transmission_interface/SimpleTransmission</type>
-  <joint name="joint2">
-    <hardwareInterface>PositionJointInterface</hardwareInterface>
-  </joint>
-  <actuator name="joint2_actr">
-    <hardwareInterface>PositionJointInterface</hardwareInterface>
-    <mechanicalReduction>1</mechanicalReduction>
-  </actuator>
-</transmission>
-<joint name="joint3" type="revolute">
-  <origin rpy="0 0 0" xyz="0.011322 -0.000113 0.2142"/>
-  <parent link="Forearm__1"/>
-  <child link="wrist_1__1"/>
-  <axis xyz="0.01 -1.7e-05 -0.0"/>
-  <limit effort="100" velocity="0.5" upper="2.27" lower="-2.27"/>
-</joint>
-<transmission name="joint3_tran">
-  <type>transmission_interface/SimpleTransmission</type>
-  <joint name="joint3">
-    <hardwareInterface>PositionJointInterface</hardwareInterface>
-  </joint>
-  <actuator name="joint3_actr">
-    <hardwareInterface>PositionJointInterface</hardwareInterface>
-    <mechanicalReduction>1</mechanicalReduction>
-  </actuator>
-</transmission>
-<joint name="joint1" type="revolute">
-  <origin rpy="0 0 0" xyz="0.065458 5e-06 0.03505"/>
-  <parent link="shoulder__1"/>
-  <child link="upper_arm__1"/>
-  <axis xyz="0.01 -1.7e-05 0.0"/>
-  <limit effort="100" velocity="0.5" upper="1.57" lower="-1.57"/>
-</joint>
-<transmission name="joint1_tran">
-  <type>transmission_interface/SimpleTransmission</type>
-  <joint name="joint1">
-    <hardwareInterface>PositionJointInterface</hardwareInterface>
-  </joint>
-  <actuator name="joint1_actr">
-    <hardwareInterface>PositionJointInterface</hardwareInterface>
-    <mechanicalReduction>1</mechanicalReduction>
-  </actuator>
-</transmission>
-<joint name="joint0" type="revolute">
-  <origin rpy="0 0 0" xyz="0.000666 -0.07459 0.0302246"/>
-  <parent link="base_link"/>
-  <child link="shoulder__1"/>
-  <axis xyz="0.0 0.0 0.01"/>
-  <limit effort="100" velocity="0.5" upper="2.27" lower="-2.27"/>
-</joint>
-<transmission name="joint0_tran">
-  <type>transmission_interface/SimpleTransmission</type>
-  <joint name="joint0">
-    <hardwareInterface>PositionJointInterface</hardwareInterface>
-  </joint>
-  <actuator name="joint0_actr">
-    <hardwareInterface>PositionJointInterface</hardwareInterface>
-    <mechanicalReduction>1</mechanicalReduction>
-  </actuator>
-</transmission>
-<joint name="joint4" type="revolute">
-  <origin rpy="0 0 0" xyz="0.0441 2.6e-05 0.031555"/>
-  <!-- <origin rpy="0 0 0" xyz="0.0267067 2.6e-05 0.030455"/> -->
-  <parent link="wrist_1__1"/>
-  <child link="wrist_2__1"/>
-  <axis xyz="0.0 2.2e-05 0.01"/>
-  <limit effort="100" velocity="0.5" upper="2.27" lower="-2.27"/>
-</joint>
-<transmission name="joint4_tran">
-  <type>transmission_interface/SimpleTransmission</type>
-  <joint name="joint4">
-    <hardwareInterface>PositionJointInterface</hardwareInterface>
-  </joint>
-  <actuator name="joint4_actr">
-    <hardwareInterface>PositionJointInterface</hardwareInterface>
-    <mechanicalReduction>1</mechanicalReduction>
-  </actuator>
-</transmission>
-<joint name="joint5" type="revolute">
-  <origin rpy="0 0 0" xyz="-0.000148 0.031513 -0.1089"/>
-  <parent link="wrist_2__1"/>
-  <child link="end_effector_link__1"/>
-  <axis xyz="-4.7e-05 0.01 -2.2e-05"/>
-  <limit effort="100" velocity="0.5" upper="2.27" lower="-2.27"/>
-</joint>
-<transmission name="joint5_tran">
-  <type>transmission_interface/SimpleTransmission</type>
-  <joint name="joint5">
-    <hardwareInterface>PositionJointInterface</hardwareInterface>
-  </joint>
-  <actuator name="joint5_actr">
-    <hardwareInterface>PositionJointInterface</hardwareInterface>
-    <mechanicalReduction>1</mechanicalReduction>
-  </actuator>
-</transmission>
-<gazebo>
-  <plugin filename="libgazebo_ros_control.so" name="control"/>
-</gazebo>
-</robot>
+<?xml version="1.0"?>
+<robot xmlns:xacro="https://www.ros.org/wiki/xacro" name="we_r2_arm">
+    <link name="world" />
+    <link name="base_link">
+        <visual>
+            <origin rpy="0 0 0"  xyz="0 0 0" />
+            <geometry>
+                <mesh filename="package://we_r2_arm_description/meshes/shoulder_actuator_1.stl" scale="1 1 1" />
+            </geometry>
+        </visual>
+    </link>
+    <joint name="virtual_joint" type="fixed">
+        <parent link="world" />
+        <child link="base_link" />
+        <origin rpy="0 0 0" xyz="0 0 0" />
+    </joint>
+</robot>`
