Commit message: feat: implement the low part of the urdf model

File: src/we_r2_arm_description/urdf/we_r2_arm.urdf.xacro (robot description, xacro)
@@ -1,17 +1,50 @@
 <?xml version="1.0"?>
 <robot xmlns:xacro="https://www.ros.org/wiki/xacro" name="we_r2_arm">
-    <link name="world" />
-    <link name="base_link">
-        <visual>
-            <origin rpy="0 0 0"  xyz="0 0 0" />
-            <geometry>
-                <mesh filename="package://we_r2_arm_description/meshes/shoulder_actuator_1.stl" scale="1 1 1" />
-            </geometry>
-        </visual>
-    </link>
-    <joint name="virtual_joint" type="fixed">
-        <parent link="world" />
-        <child link="base_link" />
-        <origin rpy="0 0 0" xyz="0 0 0" />
-    </joint>
-</robot>`
+  <xacro:property name="PI" value="3.14159" />
+  <xacro:property name="effort" value="100.0" />
+  <xacro:property name="velocity" value="0.5" />
+  <link name="world" />
+  <link name="base_link">
+      <visual>
+          <origin rpy="0 0 0"  xyz="0 0 0" />
+          <geometry>
+            <mesh filename="package://we_r2_arm_description/meshes/basement.stl" scale="1 1 1" />
+          </geometry>
+      </visual>
+  </link>
+  <link name="shoulder_1">
+    <visual>
+      <origin rpy="0 0 0"  xyz="0 0 -0.09" />
+          <geometry>
+            <mesh filename="package://we_r2_arm_description/meshes/1.stl" scale="1 1 1" />
+          </geometry>
+    </visual>
+  </link>
+  <link name="shoulder_2">
+    <visual>
+      <origin rpy="0 0 0"  xyz="0 0 -0.1225" />
+          <geometry>
+            <mesh filename="package://we_r2_arm_description/meshes/2.stl" scale="1 1 1" />
+          </geometry>
+    </visual>
+  </link>
+  <joint name="virtual_joint" type="fixed">
+    <parent link="world" />
+    <child link="base_link" />
+    <origin rpy="0 0 0" xyz="0 0 0" />
+  </joint>
+  <joint name="joint_0" type="revolute">
+    <parent link="base_link" />
+    <child link="shoulder_1" />
+    <origin rpy="0 0 0" xyz="0 0 0.09" />
+    <axis xyz="0 0 1" />
+    <limit lower="-${PI/2}" upper="${PI/2}" effort="${effort}" velocity="${velocity}" />
+  </joint>
+  <joint name="joint_1" type="revolute">
+    <parent link="shoulder_1" />
+    <child link="shoulder_2" />
+    <origin rpy="0 0 0" xyz="0 0 0.0375" />
+    <axis xyz="1 0 0" />
+    <limit lower="-${PI/2}" upper="${PI/2}" effort="${effort}" velocity="${velocity}" />
+  </joint>
+</robot>

Commit message: feat: add an arm and another shoulder

File: src/we_r2_arm_description/urdf/we_r2_arm.urdf.xacro (robot description, xacro)
@@ -23,7 +23,23 @@
   <link name="shoulder_2">
     <visual>
-      <origin rpy="0 0 0"  xyz="0 0 -0.1225" />
+      <origin rpy="0 0 0"  xyz="-0.0925 0 -0.1225" />
           <geometry>
             <mesh filename="package://we_r2_arm_description/meshes/2.stl" scale="1 1 1" />
+          </geometry>
+    </visual>
+  </link>
+  <link name="arm_1">
+    <visual>
+      <origin rpy="0 0 0"  xyz="-0.0925 0 -0.238" />
+          <geometry>
+            <mesh filename="package://we_r2_arm_description/meshes/3.stl" scale="1 1 1" />
+          </geometry>
+    </visual>
+  </link>
+  <link name="shoulder_3">
+    <visual>
+      <origin rpy="0 0 0"  xyz="-0.0925 0 -0.353" />
+          <geometry>
+            <mesh filename="package://we_r2_arm_description/meshes/4.stl" scale="1 1 1" />
           </geometry>
     </visual>
@@ -44,7 +60,17 @@
     <parent link="shoulder_1" />
     <child link="shoulder_2" />
-    <origin rpy="0 0 0" xyz="0 0 0.0375" />
+    <origin rpy="0 0 0" xyz="0.0925 0 0.0375" />
     <axis xyz="1 0 0" />
     <limit lower="-${PI/2}" upper="${PI/2}" effort="${effort}" velocity="${velocity}" />
   </joint>
+  <joint name="joint_2" type="fixed">
+    <parent link="shoulder_2" />
+    <child link="arm_1" />
+    <origin rpy="0 0 0" xyz="0 0 0.115" />
+  </joint>
+  <joint name="joint_3" type="fixed">
+    <parent link="arm_1" />
+    <child link="shoulder_3" />
+    <origin rpy="0 0 0" xyz="0 0 0.115" />
+  </joint>
 </robot>

Commit message: feat: add the last arm

File: src/we_r2_arm_description/urdf/we_r2_arm.urdf.xacro (robot description, xacro)
@@ -23,5 +23,5 @@
   <link name="shoulder_2">
     <visual>
-      <origin rpy="0 0 0"  xyz="-0.0925 0 -0.1225" />
+      <origin rpy="0 0 0"  xyz="-0.0975 0 -0.1225" />
           <geometry>
             <mesh filename="package://we_r2_arm_description/meshes/2.stl" scale="1 1 1" />
@@ -31,5 +31,5 @@
   <link name="arm_1">
     <visual>
-      <origin rpy="0 0 0"  xyz="-0.0925 0 -0.238" />
+      <origin rpy="0 0 0"  xyz="-0.0975 0 -0.238" />
           <geometry>
             <mesh filename="package://we_r2_arm_description/meshes/3.stl" scale="1 1 1" />
@@ -39,7 +39,15 @@
   <link name="shoulder_3">
     <visual>
-      <origin rpy="0 0 0"  xyz="-0.0925 0 -0.353" />
+      <origin rpy="0 0 0"  xyz="-0.0975 0 -0.353" />
           <geometry>
             <mesh filename="package://we_r2_arm_description/meshes/4.stl" scale="1 1 1" />
+          </geometry>
+    </visual>
+  </link>
+  <link name="arm_2">
+    <visual>
+      <origin rpy="0 0 0"  xyz="-0.035 0 -0.353" />
+          <geometry>
+            <mesh filename="package://we_r2_arm_description/meshes/5.stl" scale="1 1 1" />
           </geometry>
     </visual>
@@ -60,5 +68,5 @@
     <parent link="shoulder_1" />
     <child link="shoulder_2" />
-    <origin rpy="0 0 0" xyz="0.0925 0 0.0375" />
+    <origin rpy="0 0 0" xyz="0.0975 0 0.0375" />
     <axis xyz="1 0 0" />
     <limit lower="-${PI/2}" upper="${PI/2}" effort="${effort}" velocity="${velocity}" />
@@ -74,3 +82,10 @@
     <origin rpy="0 0 0" xyz="0 0 0.115" />
   </joint>
+  <joint name="joint_4" type="revolute">
+    <parent link="shoulder_3" />
+    <child link="arm_2" />
+    <origin rpy="0 0 0" xyz="-0.062 0 0" />
+    <axis xyz="1 0 0" />
+    <limit lower="-${PI/2}" upper="${PI/2}" effort="${effort}" velocity="${velocity}" />
+  </joint>
 </robot>

Commit message: feat: add joint_5

File: src/we_r2_arm_description/urdf/we_r2_arm.urdf.xacro (robot description, xacro)
@@ -53,4 +53,12 @@
     </visual>
   </link>
+  <link name="wrist_1">
+    <visual>
+      <origin rpy="0 0 0"  xyz="-0.035 0 -0.5655" />
+          <geometry>
+            <mesh filename="package://we_r2_arm_description/meshes/6.stl" scale="1 1 1" />
+          </geometry>
+    </visual>
+  </link>
   <joint name="virtual_joint" type="fixed">
     <parent link="world" />
@@ -89,3 +97,10 @@
     <limit lower="-${PI/2}" upper="${PI/2}" effort="${effort}" velocity="${velocity}" />
   </joint>
+  <joint name="joint_5" type="revolute">
+    <parent link="arm_2" />
+    <child link="wrist_1" />
+    <origin rpy="0 0 0" xyz="0 0 0.2125" />
+    <axis xyz="0 0 1" />
+    <limit lower="-${PI/2}" upper="${PI/2}" effort="${effort}" velocity="${velocity}" />
+  </joint>
 </robot>

Commit message: feat: add wrist 2

File: src/we_r2_arm_description/urdf/we_r2_arm.urdf.xacro (robot description, xacro)
@@ -61,4 +61,12 @@
     </visual>
   </link>
+  <link name="wrist_2">
+    <visual>
+      <origin rpy="0 0 0"  xyz="-0.106 0 -0.5655" />
+          <geometry>
+            <mesh filename="package://we_r2_arm_description/meshes/7.stl" scale="1 1 1" />
+          </geometry>
+    </visual>
+  </link>
   <joint name="virtual_joint" type="fixed">
     <parent link="world" />
@@ -104,3 +112,10 @@
     <limit lower="-${PI/2}" upper="${PI/2}" effort="${effort}" velocity="${velocity}" />
   </joint>
+  <joint name="joint_6" type="revolute">
+    <parent link="wrist_1" />
+    <child link="wrist_2" />
+    <origin rpy="0 0 0" xyz="0.071 0 0" />
+    <axis xyz="1 0 0" />
+    <limit lower="-${PI/2}" upper="${PI/2}" effort="${effort}" velocity="${velocity}" />
+  </joint>
 </robot>

Commit message: feat: finish the main urdf structure by adding last link and joint

File: src/we_r2_arm_description/urdf/we_r2_arm.urdf.xacro (robot description, xacro)
@@ -69,4 +69,12 @@
     </visual>
   </link>
+  <link name="wrist_3">
+    <visual>
+      <origin rpy="0 0 0"  xyz="-0.106 0 -0.4955" />
+          <geometry>
+            <mesh filename="package://we_r2_arm_description/meshes/8.stl" scale="1 1 1" />
+          </geometry>
+    </visual>
+  </link>
   <joint name="virtual_joint" type="fixed">
     <parent link="world" />
@@ -119,3 +127,10 @@
     <limit lower="-${PI/2}" upper="${PI/2}" effort="${effort}" velocity="${velocity}" />
   </joint>
+  <joint name="joint_7" type="revolute">
+    <parent link="wrist_2" />
+    <child link="wrist_3" />
+    <origin rpy="0 0 0" xyz="0 0 -0.07" />
+    <axis xyz="0 0 1" />
+    <limit lower="-${PI/2}" upper="${PI/2}" effort="${effort}" velocity="${velocity}" />
+  </joint>
 </robot>

Commit message: refactor: rename links

File: src/we_r2_arm_description/urdf/we_r2_arm.urdf.xacro (robot description, xacro)
@@ -9,5 +9,5 @@
           <origin rpy="0 0 0"  xyz="0 0 0" />
           <geometry>
-            <mesh filename="package://we_r2_arm_description/meshes/basement.stl" scale="1 1 1" />
+            <mesh filename="package://we_r2_arm_description/meshes/_basement.stl" scale="1 1 1" />
           </geometry>
       </visual>
@@ -17,5 +17,5 @@
       <origin rpy="0 0 0"  xyz="0 0 -0.09" />
           <geometry>
-            <mesh filename="package://we_r2_arm_description/meshes/1.stl" scale="1 1 1" />
+            <mesh filename="package://we_r2_arm_description/meshes/_shoulder_link_1.stl" scale="1 1 1" />
           </geometry>
     </visual>
@@ -25,5 +25,5 @@
       <origin rpy="0 0 0"  xyz="-0.0975 0 -0.1225" />
           <geometry>
-            <mesh filename="package://we_r2_arm_description/meshes/2.stl" scale="1 1 1" />
+            <mesh filename="package://we_r2_arm_description/meshes/_shoulder_link_2.stl" scale="1 1 1" />
           </geometry>
     </visual>
@@ -33,5 +33,5 @@
       <origin rpy="0 0 0"  xyz="-0.0975 0 -0.238" />
           <geometry>
-            <mesh filename="package://we_r2_arm_description/meshes/3.stl" scale="1 1 1" />
+            <mesh filename="package://we_r2_arm_description/meshes/_arm_link_1.stl" scale="1 1 1" />
           </geometry>
     </visual>
@@ -41,5 +41,5 @@
       <origin rpy="0 0 0"  xyz="-0.0975 0 -0.353" />
           <geometry>
-            <mesh filename="package://we_r2_arm_description/meshes/4.stl" scale="1 1 1" />
+            <mesh filename="package://we_r2_arm_description/meshes/_shoulder_link_3.stl" scale="1 1 1" />
           </geometry>
     </visual>
@@ -49,5 +49,5 @@
       <origin rpy="0 0 0"  xyz="-0.035 0 -0.353" />
           <geometry>
-            <mesh filename="package://we_r2_arm_description/meshes/5.stl" scale="1 1 1" />
+            <mesh filename="package://we_r2_arm_description/meshes/_arm_link_2.stl" scale="1 1 1" />
           </geometry>
     </visual>
@@ -57,5 +57,5 @@
       <origin rpy="0 0 0"  xyz="-0.035 0 -0.5655" />
           <geometry>
-            <mesh filename="package://we_r2_arm_description/meshes/6.stl" scale="1 1 1" />
+            <mesh filename="package://we_r2_arm_description/meshes/_wrist_link_1.stl" scale="1 1 1" />
           </geometry>
     </visual>
@@ -65,5 +65,5 @@
       <origin rpy="0 0 0"  xyz="-0.106 0 -0.5655" />
           <geometry>
-            <mesh filename="package://we_r2_arm_description/meshes/7.stl" scale="1 1 1" />
+            <mesh filename="package://we_r2_arm_description/meshes/_wrist_link_2.stl" scale="1 1 1" />
           </geometry>
     </visual>
@@ -73,5 +73,5 @@
       <origin rpy="0 0 0"  xyz="-0.106 0 -0.4955" />
           <geometry>
-            <mesh filename="package://we_r2_arm_description/meshes/8.stl" scale="1 1 1" />
+            <mesh filename="package://we_r2_arm_description/meshes/_wrist_link_3.stl" scale="1 1 1" />
           </geometry>
     </visual>

Commit message: refactor: change joints' names

File: src/we_r2_arm_description/urdf/we_r2_arm.urdf.xacro (robot description, xacro)
@@ -96,15 +96,15 @@
     <limit lower="-${PI/2}" upper="${PI/2}" effort="${effort}" velocity="${velocity}" />
   </joint>
-  <joint name="joint_2" type="fixed">
+  <joint name="fix_s2_a1" type="fixed">
     <parent link="shoulder_2" />
     <child link="arm_1" />
     <origin rpy="0 0 0" xyz="0 0 0.115" />
   </joint>
-  <joint name="joint_3" type="fixed">
+  <joint name="fix_a1_s3" type="fixed">
     <parent link="arm_1" />
     <child link="shoulder_3" />
     <origin rpy="0 0 0" xyz="0 0 0.115" />
   </joint>
-  <joint name="joint_4" type="revolute">
+  <joint name="joint_2" type="revolute">
     <parent link="shoulder_3" />
     <child link="arm_2" />
@@ -113,5 +113,5 @@
     <limit lower="-${PI/2}" upper="${PI/2}" effort="${effort}" velocity="${velocity}" />
   </joint>
-  <joint name="joint_5" type="revolute">
+  <joint name="joint_3" type="revolute">
     <parent link="arm_2" />
     <child link="wrist_1" />
@@ -120,5 +120,5 @@
     <limit lower="-${PI/2}" upper="${PI/2}" effort="${effort}" velocity="${velocity}" />
   </joint>
-  <joint name="joint_6" type="revolute">
+  <joint name="joint_4" type="revolute">
     <parent link="wrist_1" />
     <child link="wrist_2" />
@@ -127,5 +127,5 @@
     <limit lower="-${PI/2}" upper="${PI/2}" effort="${effort}" velocity="${velocity}" />
   </joint>
-  <joint name="joint_7" type="revolute">
+  <joint name="joint_5" type="revolute">
     <parent link="wrist_2" />
     <child link="wrist_3" />

Commit message: feat: add draft collision models

File: src/we_r2_arm_description/urdf/we_r2_arm.urdf.xacro (robot description, xacro)
@@ -12,68 +12,122 @@
           </geometry>
       </visual>
+      <collision>
+          <origin rpy="0 0 0"  xyz="0 0 0" />
+          <geometry>
+            <mesh filename="package://we_r2_arm_description/meshes/_basement.stl" scale="1 1 1" />
+          </geometry>
+      </collision>
   </link>
   <link name="shoulder_1">
-    <visual>
-      <origin rpy="0 0 0"  xyz="0 0 -0.09" />
+      <visual>
+          <origin rpy="0 0 0"  xyz="0 0 -0.09" />
           <geometry>
             <mesh filename="package://we_r2_arm_description/meshes/_shoulder_link_1.stl" scale="1 1 1" />
           </geometry>
-    </visual>
+      </visual>
+      <collision>
+          <origin rpy="0 0 0"  xyz="0 0 -0.09" />
+          <geometry>
+            <mesh filename="package://we_r2_arm_description/meshes/_shoulder_link_1.stl" scale="1 1 1" />
+          </geometry>
+      </collision>
   </link>
   <link name="shoulder_2">
-    <visual>
-      <origin rpy="0 0 0"  xyz="-0.0975 0 -0.1225" />
+      <visual>
+          <origin rpy="0 0 0"  xyz="-0.0975 0 -0.1225" />
           <geometry>
             <mesh filename="package://we_r2_arm_description/meshes/_shoulder_link_2.stl" scale="1 1 1" />
           </geometry>
-    </visual>
+      </visual>
+      <collision>
+          <origin rpy="0 0 0"  xyz="-0.0975 0 -0.1225" />
+          <geometry>
+            <mesh filename="package://we_r2_arm_description/meshes/_shoulder_link_2.stl" scale="1 1 1" />
+          </geometry>
+      </collision>
   </link>
   <link name="arm_1">
-    <visual>
-      <origin rpy="0 0 0"  xyz="-0.0975 0 -0.238" />
+      <visual>
+          <origin rpy="0 0 0"  xyz="-0.0975 0 -0.238" />
           <geometry>
             <mesh filename="package://we_r2_arm_description/meshes/_arm_link_1.stl" scale="1 1 1" />
           </geometry>
-    </visual>
+      </visual>
+      <collision>
+          <origin rpy="0 0 0"  xyz="-0.0975 0 -0.238" />
+          <geometry>
+            <mesh filename="package://we_r2_arm_description/meshes/_arm_link_1.stl" scale="1 1 1" />
+          </geometry>
+      </collision>
   </link>
   <link name="shoulder_3">
-    <visual>
-      <origin rpy="0 0 0"  xyz="-0.0975 0 -0.353" />
+      <visual>
+          <origin rpy="0 0 0"  xyz="-0.0975 0 -0.353" />
           <geometry>
             <mesh filename="package://we_r2_arm_description/meshes/_shoulder_link_3.stl" scale="1 1 1" />
           </geometry>
-    </visual>
+      </visual>
+      <collision>
+          <origin rpy="0 0 0"  xyz="-0.0975 0 -0.353" />
+          <geometry>
+            <mesh filename="package://we_r2_arm_description/meshes/_shoulder_link_3.stl" scale="1 1 1" />
+          </geometry>
+      </collision>
   </link>
   <link name="arm_2">
-    <visual>
-      <origin rpy="0 0 0"  xyz="-0.035 0 -0.353" />
+      <visual>
+          <origin rpy="0 0 0"  xyz="-0.035 0 -0.353" />
           <geometry>
             <mesh filename="package://we_r2_arm_description/meshes/_arm_link_2.stl" scale="1 1 1" />
           </geometry>
-    </visual>
+      </visual>
+      <collision>
+          <origin rpy="0 0 0"  xyz="-0.035 0 -0.353" />
+          <geometry>
+            <mesh filename="package://we_r2_arm_description/meshes/_arm_link_2.stl" scale="1 1 1" />
+          </geometry>
+      </collision>
   </link>
   <link name="wrist_1">
-    <visual>
-      <origin rpy="0 0 0"  xyz="-0.035 0 -0.5655" />
+      <visual>
+          <origin rpy="0 0 0"  xyz="-0.035 0 -0.5655" />
           <geometry>
             <mesh filename="package://we_r2_arm_description/meshes/_wrist_link_1.stl" scale="1 1 1" />
           </geometry>
-    </visual>
+      </visual>
+      <collision>
+          <origin rpy="0 0 0"  xyz="-0.035 0 -0.5655" />
+          <geometry>
+            <mesh filename="package://we_r2_arm_description/meshes/_wrist_link_1.stl" scale="1 1 1" />
+          </geometry>
+      </collision>
   </link>
   <link name="wrist_2">
-    <visual>
-      <origin rpy="0 0 0"  xyz="-0.106 0 -0.5655" />
+      <visual>
+          <origin rpy="0 0 0"  xyz="-0.106 0 -0.5655" />
           <geometry>
             <mesh filename="package://we_r2_arm_description/meshes/_wrist_link_2.stl" scale="1 1 1" />
           </geometry>
-    </visual>
+      </visual>
+      <collision>
+          <origin rpy="0 0 0"  xyz="-0.106 0 -0.5655" />
+          <geometry>
+            <mesh filename="package://we_r2_arm_description/meshes/_wrist_link_2.stl" scale="1 1 1" />
+          </geometry>
+      </collision>
   </link>
   <link name="wrist_3">
-    <visual>
-      <origin rpy="0 0 0"  xyz="-0.106 0 -0.4955" />
+      <visual>
+          <origin rpy="0 0 0"  xyz="-0.106 0 -0.4955" />
           <geometry>
             <mesh filename="package://we_r2_arm_description/meshes/_wrist_link_3.stl" scale="1 1 1" />
           </geometry>
-    </visual>
+      </visual>
+      <collision>
+          <origin rpy="0 0 0"  xyz="-0.106 0 -0.4955" />
+          <geometry>
+            <mesh filename="package://we_r2_arm_description/meshes/_wrist_link_3.stl" scale="1 1 1" />
+          </geometry>
+      </collision>
   </link>
   <joint name="virtual_joint" type="fixed">

Commit message: feat: apply preliminary inertia and mass

File: src/we_r2_arm_description/urdf/we_r2_arm.urdf.xacro (robot description, xacro)
@@ -4,6 +4,13 @@
   <xacro:property name="effort" value="100.0" />
   <xacro:property name="velocity" value="0.5" />
+  <xacro:macro name="set_inertial_properties" params="mass ixx iyy izz ixy ixz iyz">
+      <inertial>
+          <mass value="${mass}" />
+          <inertia ixx="${ixx}" ixy="${ixy}" ixz="${ixz}" iyy="${iyy}" iyz="${iyz}" izz="${izz}" />
+      </inertial>
+  </xacro:macro>
   <link name="world" />
   <link name="base_link">
+      <xacro:set_inertial_properties mass="5.4" ixx="0.02" iyy="0.02" izz="0.02" ixy="0.0" ixz="0.0" iyz="0.0" />
       <visual>
           <origin rpy="0 0 0"  xyz="0 0 0" />
@@ -20,4 +27,5 @@
   </link>
   <link name="shoulder_1">
+      <xacro:set_inertial_properties mass="5.4" ixx="0.02" iyy="0.02" izz="0.02" ixy="0.0" ixz="0.0" iyz="0.0" />
       <visual>
           <origin rpy="0 0 0"  xyz="0 0 -0.09" />
@@ -34,4 +42,5 @@
   </link>
   <link name="shoulder_2">
+      <xacro:set_inertial_properties mass="5.4" ixx="0.02" iyy="0.02" izz="0.02" ixy="0.0" ixz="0.0" iyz="0.0" />
       <visual>
           <origin rpy="0 0 0"  xyz="-0.0975 0 -0.1225" />
@@ -48,4 +57,5 @@
   </link>
   <link name="arm_1">
+      <xacro:set_inertial_properties mass="5.4" ixx="0.02" iyy="0.02" izz="0.02" ixy="0.0" ixz="0.0" iyz="0.0" />
       <visual>
           <origin rpy="0 0 0"  xyz="-0.0975 0 -0.238" />
@@ -62,4 +72,5 @@
   </link>
   <link name="shoulder_3">
+      <xacro:set_inertial_properties mass="5.4" ixx="0.02" iyy="0.02" izz="0.02" ixy="0.0" ixz="0.0" iyz="0.0" />
       <visual>
           <origin rpy="0 0 0"  xyz="-0.0975 0 -0.353" />
@@ -76,4 +87,5 @@
   </link>
   <link name="arm_2">
+      <xacro:set_inertial_properties mass="5.4" ixx="0.02" iyy="0.02" izz="0.02" ixy="0.0" ixz="0.0" iyz="0.0" />
       <visual>
           <origin rpy="0 0 0"  xyz="-0.035 0 -0.353" />
@@ -90,4 +102,5 @@
   </link>
   <link name="wrist_1">
+      <xacro:set_inertial_properties mass="5.4" ixx="0.02" iyy="0.02" izz="0.02" ixy="0.0" ixz="0.0" iyz="0.0" />
       <visual>
           <origin rpy="0 0 0"  xyz="-0.035 0 -0.5655" />
@@ -104,4 +117,5 @@
   </link>
   <link name="wrist_2">
+      <xacro:set_inertial_properties mass="5.4" ixx="0.02" iyy="0.02" izz="0.02" ixy="0.0" ixz="0.0" iyz="0.0" />
       <visual>
           <origin rpy="0 0 0"  xyz="-0.106 0 -0.5655" />
@@ -118,4 +132,5 @@
   </link>
   <link name="wrist_3">
+      <xacro:set_inertial_properties mass="5.4" ixx="0.02" iyy="0.02" izz="0.02" ixy="0.0" ixz="0.0" iyz="0.0" />
       <visual>
           <origin rpy="0 0 0"  xyz="-0.106 0 -0.4955" />

Commit message: fix: one of the joints to fixed type

File: src/we_r2_arm_description/urdf/we_r2_arm.urdf.xacro (robot description, xacro)
@@ -256,12 +256,10 @@
     <limit lower="-${PI/2}" upper="${PI/2}" effort="${effort}" velocity="${velocity}" />
   </joint>
-  <joint name="joint_3" type="revolute">
+  <joint name="fix_a2_w1" type="fixed">
     <parent link="arm_2" />
     <child link="wrist_1" />
     <origin rpy="0 0 0" xyz="0 0 0.2125" />
-    <axis xyz="0 0 1" />
-    <limit lower="-${PI/2}" upper="${PI/2}" effort="${effort}" velocity="${velocity}" />
-  </joint>
-  <joint name="joint_4" type="revolute">
+  </joint>
+  <joint name="joint_3" type="revolute">
     <parent link="wrist_1" />
     <child link="wrist_2" />
@@ -270,5 +268,5 @@
     <limit lower="-${PI/2}" upper="${PI/2}" effort="${effort}" velocity="${velocity}" />
   </joint>
-  <joint name="joint_5" type="revolute">
+  <joint name="joint_4" type="revolute">
     <parent link="wrist_2" />
     <child link="wrist_3" />

File: src/we_r2_arm_description/urdf/we_r2_arm_ros2_control.xacro (robot description, xacro)
@@ -41,11 +41,4 @@
             <state_interface name="position" />
         </joint>
-        <joint name="joint_5">
-            <command_interface name="position">
-                <param name="min">-${PI / 2}</param>
-                <param name="max">${PI / 2}</param>
-            </command_interface>
-            <state_interface name="position" />
-        </joint>
     </ros2_control>
 </robot>
